File: SDVX-aux-board/SDVX-aux-board.kicad_pcb (KiCad board)
At the start: 2 copper layers, 35 x 35 mm, 6 parts, among them CN1 AudioJack4_SwitchTR1, CN2 Conn_01x04

Commit message: Update to working design (kicad 8.0)
Connections:
- net /GND renamed GND
- net /SENS renamed SENS
- CN1 pad R1: /R -> R
- CN1 pad T: /L -> L
- CN2 pad 1: /L -> R
- CN2 pad 2: /R -> L
Routing:
- net /L: track 27.7 -> 0.00 mm
- net L: track 0.00 -> 18.9 mm
- net /R: track 15.7 -> 0.00 mm
- net R: track 0.00 -> 14.2 mm
Other:
- board text added: "Designed by VeyPatch"
- board text removed: "Designed by patchii"
